Commit message: added laser_frame update to xacro file

File: amr_description/xacro/ld250.urdf.xacro (robot description, xacro)
@@ -1,40 +1,68 @@
 <?xml version="1.0"?>
 <robot xmlns:xacro="http://www.ros.org/wiki/xacro" name="ld250_lib">
-<xacro:macro name="ld250" params="prefix:='' parent:='' xyz:='0 0 0' rpy:='0 0 0' mesh_pkg:='amr_description'">
-<material name="${prefix}blue"><color rgba="0 0 0.8 1"/></material>
-<material name="${prefix}black"><color rgba="0 0 0 1"/></material>
-<material name="${prefix}white"><color rgba="1 1 1 1"/></material>
-<link name="${prefix}base_link"/>
-<link name="${prefix}main_body">
-  <visual>
-    <origin rpy="0 0 3.141582654" xyz="0 0 0"/>
-    <geometry>
-      <mesh filename="package://${mesh_pkg}/meshes/LD250.obj"/>
-    </geometry>
-    <material name="${prefix}white"/>
-  </visual>
-  <collision>
-    <origin rpy="0 0 3.141592654" xyz="0 0 0"/>
-    <geometry>
-      <mesh filename="package://${mesh_pkg}/meshes/LD250.obj"/>
-    </geometry>
-  </collision>
-  <inertial>
-    <mass value="4.07"/>
-    <inertia ixx="0.426" ixy="0.0" ixz="0.0" iyy="0.496" iyz="0.0" izz="0.91"/>
-  </inertial>
-</link>
-<joint name="${prefix}main_body_to_base" type="fixed">
-  <parent link="${prefix}base_link"/>
-  <child link="${prefix}main_body"/>
-  <origin xyz="0 0 0"/>
-</joint>
-<xacro:if value="${parent != ''}">
-  <joint name="${prefix}base_mount" type="fixed">
-    <parent link="${parent}"/>
-    <child link="${prefix}base_link"/>
-    <origin xyz="${xyz}" rpy="${rpy}"/>
-  </joint>
-</xacro:if>
+  <!--
+    Updated to match LD250.urdf:
+    - Adds laser_frame link
+    - Adds base_link_to_laser_frame fixed joint at xyz="0.45 0 0.195"
+    - Keeps main_body mesh, inertial, and fixed joints
+  -->
+  <xacro:macro name="ld250" params="prefix:='' parent:='' xyz:='0 0 0' rpy:='0 0 0' mesh_pkg:='amr_description'">
+    <!-- Materials (prefixed to avoid name collisions when instantiating multiple robots) -->
+    <material name="${prefix}blue"><color rgba="0 0 0.8 1"/></material>
+    <material name="${prefix}black"><color rgba="0 0 0 1"/></material>
+    <material name="${prefix}white"><color rgba="1 1 1 1"/></material>
+    <!-- Base link -->
+    <link name="${prefix}base_link"/>
+    <!-- Main body with mesh -->
+    <link name="${prefix}main_body">
+      <visual>
+        <origin rpy="0 0 3.141582654" xyz="0 0 0"/>
+        <geometry>
+          <mesh filename="package://${mesh_pkg}/meshes/LD250.obj"/>
+        </geometry>
+        <material name="${prefix}white"/>
+      </visual>
+      <collision>
+        <origin rpy="0 0 3.141592654" xyz="0 0 0"/>
+        <geometry>
+          <mesh filename="package://${mesh_pkg}/meshes/LD250.obj"/>
+        </geometry>
+      </collision>
+      <inertial>
+        <mass value="4.07"/>
+        <inertia ixx="0.426" ixy="0.0" ixz="0.0" iyy="0.496" iyz="0.0" izz="0.91"/>
+      </inertial>
+    </link>
+    <!-- Base to main body fixed joint -->
+    <joint name="${prefix}main_body_to_base" type="fixed">
+      <parent link="${prefix}base_link"/>
+      <child link="${prefix}main_body"/>
+      <origin xyz="0 0 0"/>
+    </joint>
+    <!-- Laser frame -->
+    <link name="${prefix}laser_frame"/>
+    <!-- Base to laser frame fixed joint (matches LD250.urdf) -->
+    <joint name="${prefix}base_link_to_laser_frame" type="fixed">
+      <parent link="${prefix}base_link"/>
+      <child link="${prefix}laser_frame"/>
+      <origin xyz="0.45 0 0.195"/>
+    </joint>
+    <!-- Optional mounting to an external parent -->
+    <xacro:if value="${parent != ''}">
+      <joint name="${prefix}base_mount" type="fixed">
+        <parent link="${parent}"/>
+        <child link="${prefix}base_link"/>
+        <origin xyz="${xyz}" rpy="${rpy}"/>
+      </joint>
+    </xacro:if>
+    <!--
+      Dimensions (from LD250.urdf comments):
+      - length: 950 mm
+      - width: 696 mm
+      - laser glass offset front: 20 mm
+      - laser glass offset back: 120 mm
+      - laser glass bottom height: 180 mm
+      - laser glass top height: 210 mm
+    -->
   </xacro:macro>
 </robot>

Commit message: optimized launch files

File: amr_description/xacro/ld250.urdf.xacro (robot description, xacro)
@@ -13,5 +13,6 @@
     <material name="${prefix}white"><color rgba="1 1 1 1"/></material>
     <!-- Base link -->
-    <link name="${prefix}base_link"/>
+    <link name="${prefix}base_link">
+    </link>
     <!-- Main body with mesh -->
     <link name="${prefix}main_body">
@@ -42,4 +43,5 @@
     <!-- Laser frame -->
     <link name="${prefix}laser_frame"/>
+    </link>
     <!-- Base to laser frame fixed joint (matches LD250.urdf) -->
     <joint name="${prefix}base_link_to_laser_frame" type="fixed">

Commit message: optimized launch files

File: amr_description/xacro/ld250.urdf.xacro (robot description, xacro)
@@ -42,5 +42,5 @@
     </joint>
     <!-- Laser frame -->
-    <link name="${prefix}laser_frame"/>
+    <link name="${prefix}laser_frame">
     </link>
     <!-- Base to laser frame fixed joint (matches LD250.urdf) -->

Commit message: minor change to xacro file link names

File: amr_description/xacro/ld250.urdf.xacro (robot description, xacro)
@@ -5,5 +5,5 @@
     - Adds laser_frame link
     - Adds base_link_to_laser_frame fixed joint at xyz="0.45 0 0.195"
-    - Keeps main_body mesh, inertial, and fixed joints
+    - Keeps amr_base mesh, inertial, and fixed joints
   -->
   <xacro:macro name="ld250" params="prefix:='' parent:='' xyz:='0 0 0' rpy:='0 0 0' mesh_pkg:='amr_description'">
@@ -16,5 +16,5 @@
     </link>
     <!-- Main body with mesh -->
-    <link name="${prefix}main_body">
+    <link name="${prefix}amr_base">
       <visual>
         <origin rpy="0 0 3.141582654" xyz="0 0 0"/>
@@ -22,5 +22,7 @@
           <mesh filename="package://${mesh_pkg}/meshes/LD250.obj"/>
         </geometry>
-        <material name="${prefix}white"/>
+        <material name="grey">
+          <color rgba="0.5 0.5 0.5 1.0"/>
+        </material>
       </visual>
       <collision>
@@ -35,8 +37,8 @@
       </inertial>
     </link>
-    <!-- Base to main body fixed joint -->
-    <joint name="${prefix}main_body_to_base" type="fixed">
+    <!-- Base link to main body fixed joint -->
+    <joint name="${prefix}amr_base_to_base_link" type="fixed">
       <parent link="${prefix}base_link"/>
-      <child link="${prefix}main_body"/>
+      <child link="${prefix}amr_base"/>
       <origin xyz="0 0 0"/>
     </joint>

Commit message: updated urdf xacro models, rviz files and launch files

File: amr_description/xacro/ld250.urdf.xacro (robot description, xacro)
@@ -50,5 +50,5 @@
       <parent link="${prefix}base_link"/>
       <child link="${prefix}laser_frame"/>
-      <origin xyz="0.45 0 0.195"/>
+      <origin xyz="0.40 0 0.190"/>
     </joint>
     <!-- Optional mounting to an external parent -->
@@ -61,12 +61,14 @@
     </xacro:if>
     <!--
-      Dimensions (from LD250.urdf comments):
-      - length: 950 mm
-      - width: 696 mm
-      - base height: 340 mm
-      - laser glass offset front: 20 mm
-      - laser glass offset back: 120 mm
-      - laser glass bottom height: 180 mm
-      - laser glass top height: 210 mm
+      Dimensions (from https://files.omron.eu/downloads/latest/datasheet/en/i828_ld-series_mobile_robot_datasheet_en.pdf?v=2):
+      - length: 970 mm
+      - width: 720 mm
+      - base height: 380 mm
+      - laser glass center height: 190 mm
+      Dimensions roughly measured
+      - laser glass offset front: 35 mm
+      - laser glass offset back: 135 mm
+      Calaculated from the above dimensions:
+      - laser center from the middle of the robot: (970/2 - 135 + (135-35)/2) mm = 400 mm
     -->
   </xacro:macro>

File: amr_description/xacro/ld90.urdf.xacro (robot description, xacro)
@@ -25,8 +25,17 @@
   </inertial>
 </link>
-<joint name="${prefix}main_body_to_base" type="fixed">
+<joint name="${prefix}main_body_to_base_link" type="fixed">
   <parent link="${prefix}base_link"/>
   <child link="${prefix}main_body"/>
   <origin xyz="0 0 0"/>
+</joint>
+<!-- Laser frame -->
+<link name="${prefix}laser_frame">
+</link>
+<!-- Base to laser frame fixed joint (matches LD250.urdf) -->
+<joint name="${prefix}base_link_to_laser_frame" type="fixed">
+  <parent link="${prefix}base_link"/>
+  <child link="${prefix}laser_frame"/>
+  <origin xyz="0.265 0 0.195"/>
 </joint>
 <xacro:if value="${parent != ''}">
@@ -37,4 +46,16 @@
   </joint>
 </xacro:if>
+<!--
+  Dimensions (from https://files.omron.eu/downloads/latest/datasheet/en/i828_ld-series_mobile_robot_datasheet_en.pdf?v=2):
+  - length: 700 mm
+  - width: 500 mm
+  - base height: 380 mm
+  - laser glass center height: 190 mm
+  Dimensions roughly measured
+  - laser glass offset front: 35 mm
+  - laser glass offset back: 135 mm
+  Calaculated from the above dimensions:
+  - laser center from the middle of the robot: (700/2 - 135 + (135-35)/2) mm = 265 mm
+-->
 </xacro:macro>
 </robot>

Commit message: wip

File: amr_description/xacro/ld250.urdf.xacro (robot description, xacro)
@@ -52,4 +52,13 @@
       <origin xyz="0.40 0 0.190"/>
     </joint>
+    <!-- Laser frame -->
+    <link name="${prefix}laser_frame_low">
+    </link>
+    <!-- Base to laser frame fixed joint (matches LD250.urdf) -->
+    <joint name="${prefix}base_link_to_laser_frame_low" type="fixed">
+      <parent link="${prefix}base_link"/>
+      <child link="${prefix}laser_frame_low"/>
+      <origin xyz="0.40 0 0.060"/>
+    </joint>
     <!-- Optional mounting to an external parent -->
     <xacro:if value="${parent != ''}">
@@ -69,4 +78,5 @@
       - laser glass offset front: 35 mm
       - laser glass offset back: 135 mm
+      - lower laser glass center height: 60 mm
       Calaculated from the above dimensions:
       - laser center from the middle of the robot: (970/2 - 135 + (135-35)/2) mm = 400 mm

File: amr_description/xacro/ld90.urdf.xacro (robot description, xacro)
@@ -39,4 +39,13 @@
   <origin xyz="0.265 0 0.195"/>
 </joint>
+<!-- Laser frame -->
+<link name="${prefix}laser_frame_low">
+</link>
+<!-- Base to laser frame fixed joint (matches LD250.urdf) -->
+<joint name="${prefix}base_link_to_laser_frame_low" type="fixed">
+  <parent link="${prefix}base_link"/>
+  <child link="${prefix}laser_frame_low"/>
+  <origin xyz="0.265 0 0.195"/>
+</joint>
 <xacro:if value="${parent != ''}">
   <joint name="${prefix}base_mount" type="fixed">
@@ -55,4 +64,5 @@
   - laser glass offset front: 35 mm
   - laser glass offset back: 135 mm
+  - lower laser glass center height: 60 mm
   Calaculated from the above dimensions:
   - laser center from the middle of the robot: (700/2 - 135 + (135-35)/2) mm = 265 mm

Commit message: minor fix

File: amr_description/xacro/ld250.urdf.xacro (robot description, xacro)
@@ -7,5 +7,5 @@
     - Keeps amr_base mesh, inertial, and fixed joints
   -->
-  <xacro:macro name="ld250" params="prefix:='' parent:='' xyz:='0 0 0' rpy:='0 0 0' mesh_pkg:='amr_description'">
+  <xacro:macro name="ld250" params="prefix:='' laser_frame_name:='laser_frame' parent:='' xyz:='0 0 0' rpy:='0 0 0' mesh_pkg:='amr_description'">
     <!-- Materials (prefixed to avoid name collisions when instantiating multiple robots) -->
     <material name="${prefix}blue"><color rgba="0 0 0.8 1"/></material>
@@ -49,5 +49,5 @@
     <joint name="${prefix}base_link_to_laser_frame" type="fixed">
       <parent link="${prefix}base_link"/>
-      <child link="${prefix}laser_frame"/>
+      <child link="${prefix}${laser_frame_name}"/>
       <origin xyz="0.40 0 0.190"/>
     </joint>
@@ -58,5 +58,5 @@
     <joint name="${prefix}base_link_to_laser_frame_low" type="fixed">
       <parent link="${prefix}base_link"/>
-      <child link="${prefix}laser_frame_low"/>
+      <child link="${prefix}${laser_frame_name}_low"/>
       <origin xyz="0.40 0 0.060"/>
     </joint>

Commit message: minor change

File: amr_description/xacro/ld250.urdf.xacro (robot description, xacro)
@@ -7,5 +7,5 @@
     - Keeps main_body mesh, inertial, and fixed joints
   -->
-  <xacro:macro name="ld250" params="prefix:='' parent:='' xyz:='0 0 0' rpy:='0 0 0' mesh_pkg:='amr_description'">
+  <xacro:macro name="ld250" params="prefix:='' laser_frame_name:='laser_frame' parent:='' xyz:='0 0 0' rpy:='0 0 0' mesh_pkg:='amr_description'">
     <!-- Materials (prefixed to avoid name collisions when instantiating multiple robots) -->
     <material name="${prefix}blue"><color rgba="0 0 0.8 1"/></material>
@@ -42,10 +42,10 @@
     </joint>
     <!-- Laser frame -->
-    <link name="${prefix}laser_frame">
+    <link name="${prefix}${laser_frame_name}">
     </link>
     <!-- Base to laser frame fixed joint (matches LD250.urdf) -->
     <joint name="${prefix}base_link_to_laser_frame" type="fixed">
       <parent link="${prefix}base_link"/>
-      <child link="${prefix}laser_frame"/>
+      <child link="${prefix}${laser_frame_name}"/>
       <origin xyz="0.45 0 0.195"/>
     </joint>

Commit message: restored the ld250 xacro file

File: amr_description/xacro/ld250.urdf.xacro (robot description, xacro)
@@ -7,5 +7,5 @@
     - Keeps main_body mesh, inertial, and fixed joints
   -->
-  <xacro:macro name="ld250" params="prefix:='' laser_frame_name:='laser_frame' parent:='' xyz:='0 0 0' rpy:='0 0 0' mesh_pkg:='amr_description'">
+  <xacro:macro name="ld250" params="prefix:='' parent:='' xyz:='0 0 0' rpy:='0 0 0' mesh_pkg:='amr_description'">
     <!-- Materials (prefixed to avoid name collisions when instantiating multiple robots) -->
     <material name="${prefix}blue"><color rgba="0 0 0.8 1"/></material>
@@ -42,10 +42,10 @@
     </joint>
     <!-- Laser frame -->
-    <link name="${prefix}${laser_frame_name}">
+    <link name="${prefix}laser_frame">
     </link>
     <!-- Base to laser frame fixed joint (matches LD250.urdf) -->
     <joint name="${prefix}base_link_to_laser_frame" type="fixed">
       <parent link="${prefix}base_link"/>
-      <child link="${prefix}${laser_frame_name}"/>
+      <child link="${prefix}laser_frame"/>
       <origin xyz="0.45 0 0.195"/>
     </joint>
